Commit message: 0

File: src/robot_description/urdf/finger_affine.urdf (robot description, URDF)
Before this commit: robot visual, 5 links, 4 joints
Links:
- link graber_4t_link: geometry visual mesh filename=package://robot_description/meshes/visual/14_graber_4t.stl
- link graber_r5_link: geometry visual mesh filename=package://robot_description/meshes/visual/15_graber_r5.stl
- link graber_r67_link: geometry visual mesh filename=package://robot_description/meshes/visual/16_graber_r67_aff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

File: src/robot_description/urdf/robot_ver1.urdf (robot description, URDF)
Before this commit: robot robot, 9 links, 8 joints
Joints:
- joint graber_end: origin xyz=0 0.05342048021 0.08453550906 rpy=0 0 0 -> xyz=0 0.0464378391 0.08856368951 rpy=0 0 0
- joint remote_center: origin xyz=0.14795 -0.13458 0.023 rpy=0 1.570796 -0.5635668 -> xyz=0.15866 -0.12242 0.025 rpy=0 1.570796 -0.4829326
