Commit message: “1”

File: src/robot_description/urdf/robot_ver1.urdf (robot description, URDF)
Before this commit: robot robot, 9 links, 8 joints
Joints:
- joint link1: origin xyz=0.06078 -0.029 0.25714 rpy=-1.570796 -1.745329 0 -> xyz=0.06078 -0.031 0.25714 rpy=-1.57079632679 -1.74532925199 0
- joint link3: origin xyz=0.35 0 0.077 rpy=0 0 0.61115 -> xyz=0.35 0 0.077 rpy=0 0 0.65746552922
- joint remote_center: origin xyz=0.15866 -0.12242 0.025 rpy=0 1.570796 -0.4829326 -> xyz=0.15866 -0.12242 0.025 rpy=0 1.57079632679 -0.48293260402
- joint roll1: origin xyz=0.1862 0 -0.1475 rpy=0 2.0943951 0 -> xyz=0.1862 0 -0.1475 rpy=0 2.09439510239 0
- joint roll2: origin xyz=0.15587 0 0.155 rpy=0 -0.261799 0 -> xyz=0.15587 0 0.155 rpy=0 -0.26179938779 0

File: src/robot_description/urdf/robot_ver2.urdf (robot description, URDF)
Before this commit: robot robot, 15 links, 14 joints
Links:
- link rotate2: mass 0.1 -> 0.01
Joints:
- joint child_21: limit lower=-1.57 upper=2 effort=1000.0 velocity=3.14 -> lower=-3.14 upper=3.14 effort=1000.0 velocity=3.14; origin xyz=-0.055 0 -0.36518 rpy=0 1.0471975512 0 -> xyz=-0.055 0 -0.36518 rpy=0 0 0
- joint clip21: axis 0 0 1 -> 0 1 0; origin xyz=0 0.0003 -0.0089 rpy=-1.570796 0 0 -> xyz=0 0.0003 -0.0089 rpy= 0 0 0
- joint clip22: axis 0 0 1 -> 0 1 0; origin xyz=0 -0.0003 -0.0089 rpy=1.570796 3.1415 0 -> xyz=0 -0.0003 -0.0089 rpy=0 0 0
- joint fixed: origin xyz=0 0 1 rpy=0 0 0 -> xyz=0 -0.42079 -0.41832 rpy=0 0 0.84
- joint instrument2: limit lower=-0.25 upper=0.25 effort=1000.0 velocity=3.14 -> lower=-0.5 upper=0.5 effort=1000.0 velocity=3.14; origin xyz=-0.1 0.08 0.0085 rpy=0 -1.57079632679 1.57079632679 -> xyz=-0.1 0.1 0.0085 rpy=0 -1.57079632679 1.57079632679
- joint para22: limit lower=-3 upper=3 effort=1000.0 velocity=3.14 -> lower=-6.14 upper=6.14 effort=1000.0 velocity=3.14
- joint para23: limit lower=-3 upper=3 effort=1000.0 velocity=3.14 -> lower=-6.14 upper=6.14 effort=1000.0 velocity=3.14
- joint remote_center: origin xyz=0 0 0.273205080757 rpy=1.3962634016 0 -3.1415 -> xyz= 0 0 0.273205080757 rpy=1.3962634016 0 -3.1415
- joint roll2: limit lower=-0.8 upper=0.8 effort=1000.0 velocity=3.14 -> lower=-1 upper=1 effort=1000.0 velocity=3.14
- joint roll_21: limit lower=-3 upper=3 effort=1000.0 velocity=3.14 -> lower=-6.14 upper=6.14 effort=1000.0 velocity=3.14; origin xyz=0 0 -0.15236273603 rpy=0 0 0 -> xyz=-0.13195 0 -0.07718 rpy=0 1.0472 0; type fixed -> revolute
- joint roll_22: limit lower=-3 upper=3 effort=1000.0 velocity=3.14 -> lower=-6.14 upper=6.14 effort=1000.0 velocity=3.14
- joint slide21: limit lower=-3 upper=3 effort=1000.0 velocity=3.14 -> lower=-6.14 upper=6.14 effort=1000.0 velocity=3.14
